Commit message: new robot geometry

File: description/gazebo_control.xacro (robot description, xacro)
@@ -6,5 +6,5 @@
             <left_joint>left_wheel_joint</left_joint>
             <right_joint>right_wheel_joint</right_joint>
-            <wheel_separation>0.21</wheel_separation>
+            <wheel_separation>0.41</wheel_separation>
             <wheel_diameter>0.12</wheel_diameter>
             <!-- Limits -->

File: description/lidar.xacro (robot description, xacro)
@@ -2,7 +2,7 @@
 <robot xmlns:xacro="http://www.ros.org/wiki/xacro" >
     <joint name="laser_joint" type="fixed">
-        <parent link="chassis"/>
+        <parent link="body"/>
         <child link="laser_frame"/>
-        <origin xyz="0.1 0 0.15" rpy="0 0 0"/>
+        <origin xyz="0 0 0.15" rpy="0 0 0"/>
     </joint>
     <link name="laser_frame">

File: description/robot_core.xacro (robot description, xacro)
@@ -30,23 +30,23 @@
         <parent link="base_link"/>
         <child link="chassis"/>
-        <origin xyz="-0.035 0 0"/> <!-- décalage xyz entre le référentiel chassis et le référentiel centre des roues -->
+        <origin xyz="0.045 0 -0.012"/> <!-- décalage xyz entre le référentiel chassis et le référentiel centre des roues -->
     </joint>
     <!-- Chassis size and shape-->
     <link name="chassis">
         <visual>
-            <origin xyz="0.14 0 0.01" rpy="0 0 0"/> <!-- Translation du chassis pour que les roues soient fixé en dessous -->
+            <origin xyz="-0.045 0 0.01" rpy="0 0 0"/> <!-- Translation du chassis pour que les roues soient fixé en dessous -->
             <geometry>
-                <box size="0.28 0.15 0.02"/> <!-- taille du chassis-->
+                <box size="0.09 0.35 0.005"/> <!-- taille du chassis-->
             </geometry>
             <material name="black"/> <!-- couleur du chassis-->
         </visual>
         <collision>
-            <origin xyz="0.14 0 0.01" rpy="0 0 0"/> <!-- Translation du chassis pour que les roues soient fixé en dessous -->
+            <origin xyz="-0.045 0 0.01" rpy="0 0 0"/> <!-- Translation du chassis pour que les roues soient fixé en dessous -->
             <geometry>
-                <box size="0.28 0.15 0.02"/> <!-- taille du chassis-->
+                <box size="0.09 0.35 0.005"/> <!-- taille du chassis-->
             </geometry>
         </collision>
-        <xacro:inertial_box mass="0.5" x="0.28" y="0.09" z="0.02">
-            <origin xyz="0.15 0 0.035" rpy="0 0 0"/>
+        <xacro:inertial_box mass="0.5" x="0.09" y="0.28" z="0.02">
+            <origin xyz="0.045 0 0.01" rpy="0 0 0"/>
         </xacro:inertial_box>
     </link>
@@ -56,7 +56,7 @@
     <!-- Body -->
     <joint name="body_joint" type="fixed">
-        <parent link="chassis"/>
+        <parent link="base_link"/>
         <child link="body"/>
-        <origin xyz="0.105 0 0" rpy="0 0 0"/>
+        <origin xyz="0 0.015 -0.012" rpy="0 0 0"/>
     </joint>
     <link name="body">
@@ -69,11 +69,11 @@
         </visual>
         <collision>
-            <origin xyz="0 0 0.08" rpy="0 0 0"/>
+            <origin xyz="0 0 -0.08" rpy="0 0 0"/>
             <geometry>
-                <box size="0.1 0.1 0.12"/> <!-- taille du corp-->
+                <box size="0.09 0.1 0.12"/> <!-- taille du corp-->
             </geometry>
         </collision>
-        <xacro:inertial_box mass="0.2" x="0.28" y="0.09" z="0.02">
-            <origin xyz="0.15 0 0.035" rpy="0 0 0"/>
+        <xacro:inertial_box mass="0.2" x="0.09" y="0.09" z="0.12">
+            <origin xyz="0 0 -0.08" rpy="0 0 0"/>
         </xacro:inertial_box>
     </link>
@@ -85,5 +85,5 @@
         <parent link="base_link"/>
         <child link="left_wheel"/>
-        <origin xyz="0 0.105 -0.02" rpy="-${pi/2} 0 0"/>
+        <origin xyz="0 0.205 0.02" rpy="-${pi/2} 0 0"/>
         <axis xyz="0 0 1"/>
     </joint>
@@ -111,5 +111,5 @@
         <parent link="base_link"/>
         <child link="right_wheel"/>
-        <origin xyz="0 -0.105 -0.02" rpy="${pi/2} 0 0"/>
+        <origin xyz="0 -0.205 0.02" rpy="${pi/2} 0 0"/>
         <axis xyz="0 0 -1"/>
     </joint>
@@ -137,5 +137,5 @@
         <parent link="chassis"/>
         <child link="caster_wheel"/>
-        <origin xyz="0.22 0 -0.05"/>
+        <origin xyz="-0.22 0 -0.012"/>
     </joint>
     <link name="caster_wheel">
@@ -151,5 +151,5 @@
             </geometry>
         </collision>
-        <xacro:inertial_sphere mass="0.1" radius="0.03">
+        <xacro:inertial_sphere mass="0.4" radius="0.03">
             <origin xyz="0 0 0" rpy="0 0 0"/>
         </xacro:inertial_sphere>
