Commit message: save

File: description/robot_core.xacro (robot description, xacro)
@@ -7,4 +7,7 @@
         <color rgba="1 0.3 1 1"/>
     </material>
+    <material name="purple">
+        <color rgba="0.67 0.38 0.67 1"/>
+    </material>
     <material name="blue">
         <color rgba="0.2 0.2 1 1"/>
@@ -13,6 +16,8 @@
         <color rgba="0 0 0 1"/>
     </material>
+    <!-- BASE -->
     <link name="base_link">
     </link>
+    <!-- Chassis related to the Base -->
     <joint name="chassis_joint" type ="fixed">
         <parent link="base_link"/>
@@ -20,7 +25,8 @@
         <origin xyz="-0.1 0 0"/> <!-- décalage xyz entre le référentiel chassis et le référentiel centre des roues -->
     </joint>
+    <!-- Chassis size and shape-->
     <link name="chassis">
         <visual>
-            <origin xyz="0.15 0 0.075" rpy="0 0 0"/> <!-- Translation du chassis pour que les roues soient fixé en dessous -->
+            <origin xyz="0.15 0 0.035" rpy="0 0 0"/> <!-- Translation du chassis pour que les roues soient fixé en dessous -->
             <geometry>
                 <box size="0.3 0.3 0.05"/> <!-- taille du chassis-->
@@ -29,3 +35,17 @@
         </visual>
     </link>
+    <!-- LEFT wheels link-->
+    <joint name="left_wheel_joint" type="continuous">
+        <parent link="base_link"/>
+        <child link="left_wheel"/>
+        <origin xyz=""/>
+    </joint>
+    <link name="left_wheel">
+        <visual>
+            <geometry>
+                <cylinder radius="0.05" lenght="0.04"/>
+            </geometry>
+            <material name="purple"/>
+        </visual>
+    </link>
 </robot>

Commit message: wheels

File: description/robot_core.xacro (robot description, xacro)
@@ -39,5 +39,6 @@
         <parent link="base_link"/>
         <child link="left_wheel"/>
-        <origin xyz=""/>
+        <origin xyz="0 0.175 0" rpy="-${pi/2} 0 0"/>
+        <axis xyz="0 0 1"/>
     </joint>
     <link name="left_wheel">
@@ -49,3 +50,18 @@
         </visual>
     </link>
+    <!-- right wheels link-->
+    <joint name="right_wheel_joint" type="continuous">
+        <parent link="base_link"/>
+        <child link="right_wheel"/>
+        <origin xyz="0 -0.175 0" rpy="${pi/2} 0 0"/>
+        <axis xyz="0 0 -1"/>
+    </joint>
+    <link name="right_wheel">
+        <visual>
+            <geometry>
+                <cylinder radius="0.05" lenght="0.04"/>
+            </geometry>
+            <material name="purple"/>
+        </visual>
+    </link>
 </robot>

Commit message: add collision, caster wheel, mass and inerty

File: description/robot_core.xacro (robot description, xacro)
@@ -1,4 +1,5 @@
 <?xml version="1.0"?>
 <robot xmlns:xacro="http://www.ros.org/wiki/xacro"  >
+    <xacro:include filename="inertial_macros.xacro"/>
     <material name="white">
         <color rgba="1 1 1 1"/>
@@ -6,4 +7,7 @@
     <material name="orange">
         <color rgba="1 0.3 1 1"/>
+    </material>
+    <material name="grey">
+        <color rgba="0.5 0.5 0.5 1"/>
     </material>
     <material name="purple">
@@ -34,4 +38,13 @@
             <material name="black"/> <!-- couleur du chassis-->
         </visual>
+        <collision>
+            <origin xyz="0.15 0 0.035" rpy="0 0 0"/> <!-- Translation du chassis pour que les roues soient fixé en dessous -->
+            <geometry>
+                <box size="0.3 0.3 0.05"/> <!-- taille du chassis-->
+            </geometry>
+        </collision>
+        <xacro:inertial_box mass="0.5" x="0.3" y="0.3" z="0.05">
+            <origin xyz="0.15 0 0.035" rpy="0 0 0"/>
+        </xacro:inertial_box>
     </link>
     <!-- LEFT wheels link-->
@@ -45,8 +58,16 @@
         <visual>
             <geometry>
-                <cylinder radius="0.05" lenght="0.04"/>
+                <cylinder radius="0.05" length="0.04"/>
             </geometry>
             <material name="purple"/>
         </visual>
+        <collision>
+            <geometry>
+                <cylinder radius="0.05" length="0.04"/>
+            </geometry>
+        </collision>
+        <xacro:inertial_cylinder mass="0.1" length="0.05" radius="0.05">
+            <origin xyz="0 0 0" rpy="0 0 0"/>
+        </xacro:inertial_cylinder>
     </link>
     <!-- right wheels link-->
@@ -60,8 +81,38 @@
         <visual>
             <geometry>
-                <cylinder radius="0.05" lenght="0.04"/>
+                <cylinder radius="0.05" length="0.04"/>
             </geometry>
             <material name="purple"/>
         </visual>
+        <collision>
+            <geometry>
+                <cylinder radius="0.05" length="0.04"/>
+            </geometry>
+        </collision>
+        <xacro:inertial_cylinder mass="0.1" length="0.05" radius="0.05">
+            <origin xyz="0 0 0" rpy="0 0 0"/>
+        </xacro:inertial_cylinder>
+    </link>
+        <!-- caster wheels link-->
+    <joint name="caster_wheel_joint" type="fixed">
+        <parent link="chassis"/>
+        <child link="caster_wheel"/>
+        <origin xyz="0.24 0 0"/>
+    </joint>
+    <link name="caster_wheel">
+        <visual>
+            <geometry>
+                <sphere radius="0.05"/>
+            </geometry>
+            <material name="grey"/>
+        </visual>
+        <collision>
+            <geometry>
+                <sphere radius="0.05"/>
+            </geometry>
+        </collision>
+        <xacro:inertial_sphere mass="0.1" radius="0.05">
+            <origin xyz="0 0 0" rpy="0 0 0"/>
+        </xacro:inertial_sphere>
     </link>
 </robot>

Commit message: Gazebo final init

File: description/robot_core.xacro (robot description, xacro)
@@ -12,5 +12,5 @@
     </material>
     <material name="purple">
-        <color rgba="0.67 0.38 0.67 1"/>
+        <color rgba="0.49 0.21 0.49 1"/>
     </material>
     <material name="blue">
@@ -27,30 +27,33 @@
         <parent link="base_link"/>
         <child link="chassis"/>
-        <origin xyz="-0.1 0 0"/> <!-- décalage xyz entre le référentiel chassis et le référentiel centre des roues -->
+        <origin xyz="-0.035 0 0"/> <!-- décalage xyz entre le référentiel chassis et le référentiel centre des roues -->
     </joint>
     <!-- Chassis size and shape-->
     <link name="chassis">
         <visual>
-            <origin xyz="0.15 0 0.035" rpy="0 0 0"/> <!-- Translation du chassis pour que les roues soient fixé en dessous -->
+            <origin xyz="0.14 0 0.01" rpy="0 0 0"/> <!-- Translation du chassis pour que les roues soient fixé en dessous -->
             <geometry>
-                <box size="0.3 0.3 0.05"/> <!-- taille du chassis-->
+                <box size="0.28 0.15 0.02"/> <!-- taille du chassis-->
             </geometry>
             <material name="black"/> <!-- couleur du chassis-->
         </visual>
         <collision>
-            <origin xyz="0.15 0 0.035" rpy="0 0 0"/> <!-- Translation du chassis pour que les roues soient fixé en dessous -->
+            <origin xyz="0.14 0 0.01" rpy="0 0 0"/> <!-- Translation du chassis pour que les roues soient fixé en dessous -->
             <geometry>
-                <box size="0.3 0.3 0.05"/> <!-- taille du chassis-->
+                <box size="0.28 0.15 0.02"/> <!-- taille du chassis-->
             </geometry>
         </collision>
-        <xacro:inertial_box mass="0.5" x="0.3" y="0.3" z="0.05">
+        <xacro:inertial_box mass="0.5" x="0.28" y="0.09" z="0.02">
             <origin xyz="0.15 0 0.035" rpy="0 0 0"/>
         </xacro:inertial_box>
     </link>
+    <gazebo reference="chassis">
+        <material>Gazebo/Black</material>
+    </gazebo>
     <!-- LEFT wheels link-->
     <joint name="left_wheel_joint" type="continuous">
         <parent link="base_link"/>
         <child link="left_wheel"/>
-        <origin xyz="0 0.175 0" rpy="-${pi/2} 0 0"/>
+        <origin xyz="0 0.105 -0.02" rpy="-${pi/2} 0 0"/>
         <axis xyz="0 0 1"/>
     </joint>
@@ -58,5 +61,5 @@
         <visual>
             <geometry>
-                <cylinder radius="0.05" length="0.04"/>
+                <cylinder radius="0.06" length="0.05"/>
             </geometry>
             <material name="purple"/>
@@ -64,16 +67,19 @@
         <collision>
             <geometry>
-                <cylinder radius="0.05" length="0.04"/>
+                <cylinder radius="0.06" length="0.05"/>
             </geometry>
         </collision>
-        <xacro:inertial_cylinder mass="0.1" length="0.05" radius="0.05">
+        <xacro:inertial_cylinder mass="0.1" length="0.05" radius="0.06">
             <origin xyz="0 0 0" rpy="0 0 0"/>
         </xacro:inertial_cylinder>
     </link>
+    <gazebo reference="left_wheel">
+        <material>Gazebo/Purple</material>
+    </gazebo>
     <!-- right wheels link-->
     <joint name="right_wheel_joint" type="continuous">
         <parent link="base_link"/>
         <child link="right_wheel"/>
-        <origin xyz="0 -0.175 0" rpy="${pi/2} 0 0"/>
+        <origin xyz="0 -0.105 -0.02" rpy="${pi/2} 0 0"/>
         <axis xyz="0 0 -1"/>
     </joint>
@@ -81,5 +87,5 @@
         <visual>
             <geometry>
-                <cylinder radius="0.05" length="0.04"/>
+                <cylinder radius="0.06" length="0.05"/>
             </geometry>
             <material name="purple"/>
@@ -87,21 +93,24 @@
         <collision>
             <geometry>
-                <cylinder radius="0.05" length="0.04"/>
+                <cylinder radius="0.06" length="0.05"/>
             </geometry>
         </collision>
-        <xacro:inertial_cylinder mass="0.1" length="0.05" radius="0.05">
+        <xacro:inertial_cylinder mass="0.1" length="0.05" radius="0.06">
             <origin xyz="0 0 0" rpy="0 0 0"/>
         </xacro:inertial_cylinder>
     </link>
+    <gazebo reference="right_wheel">
+        <material>Gazebo/Purple</material>
+    </gazebo>
         <!-- caster wheels link-->
     <joint name="caster_wheel_joint" type="fixed">
         <parent link="chassis"/>
         <child link="caster_wheel"/>
-        <origin xyz="0.24 0 0"/>
+        <origin xyz="0.22 0 -0.05"/>
     </joint>
     <link name="caster_wheel">
         <visual>
             <geometry>
-                <sphere radius="0.05"/>
+                <sphere radius="0.03"/>
             </geometry>
             <material name="grey"/>
@@ -109,10 +118,13 @@
         <collision>
             <geometry>
-                <sphere radius="0.05"/>
+                <sphere radius="0.03"/>
             </geometry>
         </collision>
-        <xacro:inertial_sphere mass="0.1" radius="0.05">
+        <xacro:inertial_sphere mass="0.1" radius="0.03">
             <origin xyz="0 0 0" rpy="0 0 0"/>
         </xacro:inertial_sphere>
     </link>
+    <gazebo reference="caster_wheel">
+        <material>Gazebo/Grey</material>
+    </gazebo>
 </robot>

Commit message: add body core visual

File: description/robot_core.xacro (robot description, xacro)
@@ -19,4 +19,7 @@
     <material name="black">
         <color rgba="0 0 0 1"/>
+    </material>
+    <material name="green">
+        <color rgba="0 1 0 1"/>
     </material>
     <!-- BASE -->
@@ -50,4 +53,31 @@
     <gazebo reference="chassis">
         <material>Gazebo/Black</material>
+    </gazebo>
+    <!-- Body -->
+    <joint name="body_joint" type="fixed">
+        <parent link="chassis"/>
+        <child link="body"/>
+        <origin xyz="0.105 0 0" rpy="0 0 0"/>
+    </joint>
+    <link name="body">
+        <visual>
+            <origin xyz="0 0 0.08" rpy="0 0 0"/>
+            <geometry>
+                <box size="0.1 0.1 0.12"/> <!-- taille du corp-->
+            </geometry>
+            <material name="green"/> <!-- couleur du corp-->
+        </visual>
+        <collision>
+            <origin xyz="0 0 0.08" rpy="0 0 0"/>
+            <geometry>
+                <box size="0.1 0.1 0.12"/> <!-- taille du corp-->
+            </geometry>
+        </collision>
+        <xacro:inertial_box mass="0.2" x="0.28" y="0.09" z="0.02">
+            <origin xyz="0.15 0 0.035" rpy="0 0 0"/>
+        </xacro:inertial_box>
+    </link>
+    <gazebo reference="body">
+        <material>Gazebo/Green</material>
     </gazebo>
     <!-- LEFT wheels link-->

Commit message: finish ros2control and turn wheel colision into sphere to avoid friction

File: description/robot_core.xacro (robot description, xacro)
@@ -97,5 +97,5 @@
         <collision>
             <geometry>
-                <cylinder radius="0.06" length="0.05"/>
+                <sphere radius="0.06" />
             </geometry>
         </collision>
@@ -123,5 +123,5 @@
         <collision>
             <geometry>
-                <cylinder radius="0.06" length="0.05"/>
+                <sphere radius="0.06" />
             </geometry>
         </collision>

File: description/ros2_control.xacro (robot description, xacro)
@@ -57,5 +57,5 @@
         <plugin name="gazebo_ros2_control" filename="libgazebo_ros2_control.so">
             <parameters>$(find my_bot)/config/my_controllers.yaml</parameters>
-            <parameters>$(find my_bot)/config/gaz_ros2_ctl_use_sim.yaml</parameters>
+            <!--<parameters>$(find my_bot)/config/gaz_ros2_ctl_use_sim.yaml</parameters>-->
         </plugin>
     </gazebo>

Commit message: mapper added

File: description/robot_core.xacro (robot description, xacro)
@@ -25,4 +25,12 @@
     <!-- BASE -->
     <link name="base_link">
+    </link>
+     <!-- BASE footprint SLAM -->
+    <joint name="base_footprint_joint" type="fixed">
+        <parent link="base_link"/>
+        <child link="base_footprint"/>
+        <origin xyz="0 0 0" rpy="0 0 ${pi/2}"/>
+    </joint>
+    <link name="base_footprint">
     </link>
     <!-- Chassis related to the Base -->
